File: Hardware/Dual Pi5 Connector Board/PiTrac Pi Connector.kicad_pcb (KiCad board)
At the start: 2 copper layers, 60 x 100 mm, 98 parts, among them J1 YK3210203000G, J2 YK3210203000G, J3 USB4085-GF-A, J4 USB4085-GF-A, J6 USB-A-S-RA, J7 PH1-03-UA, Q1 DMN6140L-13, Q2 DMT616MLSS-13, Q3 DMN6140L-13, Q4 DMT616MLSS-13, Q5 MMBT3904-7-F, U1 UCC2813DTR-3, U10 SN74LVC1T45DBV, U2 REF3025AIDBZR, U3 OPA357AIDBVR, U4 TS5A3157DBVR, U6 TLC555IDR, U7 SN74LVC1G08DBVR, U8 TLC555IDR, U9 SN74LVC1G17DBVR

Commit message: Update hardware documentation to correct some errors and further elaborate on some other points.
Other:
- board text added: "0.2540 mm"
- board text added: "1.6256 mm"
- board text added: "HAL lead-free"
- board text removed: "0.3000 mm"
- board text removed: "1.6000 mm"
- board text removed: "None"
